File: Hardware/PCB/LightStickAccelerometer/LightStickAccelerometer/LightStickAccelerometer.brd (EAGLE design)
At the start: 24.1 x 25.4 mm, 4 parts

Commit message: Move components to allow for some empty space on top and bottom.
Parts:
- moved J1 3.81 mm to (3.06, 6.88)
- moved R1 3.81 mm to (21.6, 19.0)
- moved R2 3.81 mm to (2.52, 19.1)
- moved J2 3.81 mm to (5.60, 25.4)
Other:
- board size 24.1 x 25.4 mm -> 24.1 x 31.7 mm
